File: stm32.kicad_sch (KiCad schematic)
At the start: 31 parts, among them J201 Conn_ST_STDC14, J203 GPIO, J204 I2C2, J205 UART1, U201 STM32G431KBT6, U202 ADXL343, Y201 16MHz

Commit message: First rev by M. FIACK
Parts:
- added R208, R209: 2K2, Resistor_SMD:R_0603_1608Metric, symbol Device:R_Small
Connections:
- net +3.3V: now also R208.1, R209.1
- net I2C2_SCL: now also R209.2
- net I2C2_SDA: now also R208.2
Other:
- moved on the sheet: J204

Commit message: TestPoint in STLink connector deleted
Parts:
- removed TP201: TestPoint, TestPoint:TestPoint_Pad_D2.0mm, symbol Connector:TestPoint
Changed lines of the file:
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@@
 	)
 	(junction
-		(at 227.33 54.61)
-		(diameter 0)
-		(color 0 0 0 0)
-	)
-	(junction
 		(at 97.79 153.67)
 		(diameter 0)
@@
 	(wire
 		(pts
-			(xy 237.49 50.8) (xy 237.49 52.07)
-		)
-		(stroke
-			(width 0)
-			(type default)
-		)
-	)
-	(wire
-		(pts
 			(xy 179.07 130.81) (xy 181.61 130.81)
 		)
@@
 	(wire
 		(pts
-			(xy 237.49 52.07) (xy 227.33 52.07)
-		)
-		(stroke
-			(width 0)
-			(type default)
-		)
-	)
-	(wire
-		(pts
 			(xy 104.14 36.83) (xy 104.14 46.99)
 		)
@@
 	(wire
 		(pts
-			(xy 227.33 54.61) (xy 228.6 54.61)
+			(xy 226.06 54.61) (xy 228.6 54.61)
 		)
 		(stroke
@@
 		)
 	)
-	(wire
-		(pts
-			(xy 226.06 54.61) (xy 227.33 54.61)
-		)
-		(stroke
-			(width 0)
-			(type default)
-		)
-	)
 	(polyline
 		(pts
@@
 	(wire
 		(pts
-			(xy 227.33 52.07) (xy 227.33 54.61)
-		)
-		(stroke
-			(width 0)
-			(type default)
-		)
-	)
-	(wire
-		(pts
 			(xy 119.38 162.56) (xy 119.38 153.67)
 		)
@@
 					(unit 1)
 				)
-			)
-		)
-	)
-	(symbol
-		(lib_id "Connector:TestPoint")
-		(at 237.49 50.8 0)
-		(unit 1)
-		(exclude_from_sim no)
-		(in_bom yes)
-		(on_board yes)
-		(dnp no)
-		(fields_autoplaced yes)
-		(property "Reference" "TP201"
-			(at 240.03 46.2279 0)
-			(effects
-				(font
-					(size 1.27 1.27)
-				)
-				(justify left)
-			)
-		)
-		(property "Value" "TestPoint"
-			(at 240.03 48.7679 0)
-			(effects
-				(font
-					(size 1.27 1.27)
-				)
-				(justify left)
-			)
-		)
-		(property "Footprint" "TestPoint:TestPoint_Pad_D2.0mm"
-			(at 242.57 50.8 0)
-			(effects
-				(font
-					(size 1.27 1.27)
-				)
-				(hide yes)
-			)
-		)
-		(property "Datasheet" "~"
-			(at 242.57 50.8 0)
-			(effects
-				(font
-					(size 1.27 1.27)
-				)
-				(hide yes)
-			)
-		)
-		(property "Description" "test point"
-			(at 237.49 50.8 0)
-			(effects
-				(font
-					(size 1.27 1.27)
-				)
-				(hide yes)
-			)
-		)
-		(pin "1"
-		)
-		(instances
-			(project ""
-				(path "/5940bb1c-61ff-4c26-9370-fcac6864aece/72bb437a-e2b3-4939-b8a1-9a9100d1fa62"
-					(reference "TP201")
-					(unit 1)
-				)

Commit message: SPI test points added
Parts:
- added CS201: CS, TestPoint:TestPoint_Pad_D2.0mm, symbol Connector:TestPoint
- added SCK201: SCK, TestPoint:TestPoint_Pad_D2.0mm, symbol Connector:TestPoint
- added SDIO201: SDIO, TestPoint:TestPoint_Pad_D2.0mm, symbol Connector:TestPoint
- INT201: renamed from TP202; value TestPoint -> INT1
- INT202: renamed from TP203; value TestPoint -> INT2
- renumbered J203 to J202, J204 to J203, J205 to J204, R209 to R203, R208 to R204, R203 to R206, R204 to R207, R207 to R208, R206 to R209
Connections:
- net CS_ACCE_SP1: now also CS201.1
- net SCK_ACCE_SPI1: now also SCK201.1
- net SDIO_ACCE_SPI1: now also SDIO201.1
Other:
- moved on the sheet: INT201, INT202, R209, U202

Commit message: +5V pin added in I2C2 connector
Parts:
- removed J203: I2C2, Connector_PinHeader_2.54mm:PinHeader_1x04_P2.54mm_Vertical, symbol Connector_Generic:Conn_01x04
- added I2C2: I2C2, Connector_PinHeader_2.54mm:PinHeader_1x05_P2.54mm_Vertical, symbol Connector_Generic:Conn_01x05
Connections:
- net +3.3V: now also I2C2.2 (Pin_2)
- net GND: now also I2C2.5 (Pin_5)
- net I2C2_SCL: now also I2C2.3 (Pin_3)
- net I2C2_SDA: now also I2C2.4 (Pin_4)
- new net +5V: I2C2.1 (Pin_1)
Changed lines of the file:
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@@
 	(text "I2C2\n"
 		(exclude_from_sim no)
-		(at 260.096 123.952 0)
+		(at 266.192 113.792 0)
 		(effects
 			(font
@@
 	(wire
 		(pts
+			(xy 257.81 128.27) (xy 257.81 130.81)
+		)
+		(stroke
+			(width 0)
+			(type default)
+		)
+	)
+	(wire
+		(pts
 			(xy 92.71 83.82) (xy 93.98 83.82)
 		)
@@
 	)
 	(symbol
-		(lib_id "Connector_Generic:Conn_01x04")
-		(at 262.89 135.89 0)
-		(unit 1)
-		(exclude_from_sim no)
-		(in_bom yes)
-		(on_board yes)
-		(dnp no)
-		(fields_autoplaced yes)
-		(property "Reference" "J203"
-			(at 265.43 135.8899 0)
-			(effects
-				(font
-					(size 1.27 1.27)
-				)
-				(justify left)
-			)
-		)
-		(property "Value" "I2C2"
-			(at 265.43 138.4299 0)
-			(effects
-				(font
-					(size 1.27 1.27)
-				)
-				(justify left)
-			)
-		)
-		(property "Footprint" "Connector_PinHeader_2.54mm:PinHeader_1x04_P2.54mm_Vertical"
-			(at 262.89 135.89 0)
-			(effects
-				(font
-					(size 1.27 1.27)
-				)
-				(hide yes)
-			)
-		)
-		(property "Datasheet" "~"
-			(at 262.89 135.89 0)
-			(effects
-				(font
-					(size 1.27 1.27)
-				)
-				(hide yes)
-			)
-		)
-		(property "Description" "Generic connector, single row, 01x04, script generated (kicad-library-utils/schlib/autogen/connector/)"
-			(at 262.89 135.89 0)
-			(effects
-				(font
-					(size 1.27 1.27)
-				)
-				(hide yes)
-			)
-		)
-		(pin "1"
-		)
-		(pin "4"
-		)
-		(pin "3"
-		)
-		(pin "2"
-		)
-		(instances
-			(project ""
-				(path "/5940bb1c-61ff-4c26-9370-fcac6864aece/72bb437a-e2b3-4939-b8a1-9a9100d1fa62"
-					(reference "J203")
-					(unit 1)
-				)
-			)
-		)
-	)
-	(symbol
 		(lib_id "Device:C")
 		(at 85.09 158.75 0)
@@
 	)
 	(symbol
+		(lib_id "Connector_Generic:Conn_01x05")
+		(at 262.89 135.89 0)
+		(unit 1)
+		(exclude_from_sim no)
+		(in_bom yes)
+		(on_board yes)
+		(dnp no)
+		(fields_autoplaced yes)
+		(property "Reference" "I2C2"
+			(at 265.43 134.6199 0)
+			(effects
+				(font
+					(size 1.27 1.27)
+				)
+				(justify left)
+			)
+		)
+		(property "Value" "I2C2"
+			(at 265.43 137.1599 0)
+			(effects
+				(font
+					(size 1.27 1.27)
+				)
+				(justify left)
+			)
+		)
+		(property "Footprint" "Connector_PinHeader_2.54mm:PinHeader_1x05_P2.54mm_Vertical"
+			(at 262.89 135.89 0)
+			(effects
+				(font
+					(size 1.27 1.27)
+				)
+				(hide yes)
+			)
+		)
+		(property "Datasheet" "~"
+			(at 262.89 135.89 0)
+			(effects
+				(font
+					(size 1.27 1.27)
+				)
+				(hide yes)
+			)
+		)
+		(property "Description" "Generic connector, single row, 01x05, script generated (kicad-library-utils/schlib/autogen/connector/)"
+			(at 262.89 135.89 0)
+			(effects
+				(font
+					(size 1.27 1.27)
+				)
+				(hide yes)
+			)
+		)
+		(pin "4"
+		)
+		(pin "2"
+		)
+		(pin "1"
+		)
+		(pin "5"
+		)
+		(pin "3"
+		)
+		(instances
+			(project ""
+				(path "/5940bb1c-61ff-4c26-9370-fcac6864aece/72bb437a-e2b3-4939-b8a1-9a9100d1fa62"
+					(reference "I2C2")
+					(unit 1)
+				)
+			)
+		)
+	)
+	(symbol
 		(lib_id "Device:Crystal_GND24_Small")
 		(at 52.07 67.31 90)
@@
 					(unit 1)
 				)
+			)
+		)
+	)
+	(symbol
+		(lib_id "power:+5V")
+		(at 257.81 128.27 0)
+		(unit 1)
+		(exclude_from_sim no)
+		(in_bom yes)
+		(on_board yes)
+		(dnp no)
+		(fields_autoplaced yes)
+		(property "Reference" "#PWR0226"
+			(at 257.81 132.08 0)
+			(effects
+				(font
+					(size 1.27 1.27)
+				)
+				(hide yes)
+			)
+		)
+		(property "Value" "+5V"
+			(at 257.81 123.19 0)
+			(effects
+				(font
+					(size 1.27 1.27)
+				)
+			)
+		)
+		(property "Footprint" ""
+			(at 257.81 128.27 0)
+			(effects
+				(font
+					(size 1.27 1.27)
+				)
+				(hide yes)
+			)
+		)
+		(property "Datasheet" ""
+			(at 257.81 128.27 0)
+			(effects
+				(font
+					(size 1.27 1.27)
+				)
+				(hide yes)
+			)
+		)
+		(property "Description" "Power symbol creates a global label with name \"+5V\""
+			(at 257.81 128.27 0)
+			(effects
+				(font
+					(size 1.27 1.27)
+				)
+				(hide yes)
+			)
+		)
+		(pin "1"
+		)
+		(instances
+			(project "tuto_kicad"
+				(path "/5940bb1c-61ff-4c26-9370-fcac6864aece/72bb437a-e2b3-4939-b8a1-9a9100d1fa62"
+					(reference "#PWR0226")
+					(unit 1)
+				)
